Commit message: Added front IR sensors, improved the visual aspect of the robot

File: prisme_description/urdf/prisme.xacro (robot description, xacro)
@@ -3,7 +3,7 @@
   <xacro:property name="PI" value="3.1415926535897931"/>
 	<!-- Fake values -->
-  <xacro:property name="mass_body" value="0.4" />
-	<xacro:property name="mass_wheel" value="0.1" />
-	<xacro:property name="mass_bpack" value="0.2" />
+  <xacro:property name="mass_body" value="0.300" />
+	<xacro:property name="mass_wheel" value="0.05" />
+	<xacro:property name="mass_bpack" value="0.4" />
 	<xacro:property name="width" value="0.0936" /> <!-- 2*46.8 = 93.6 mm -->
 	<xacro:property name="length" value="0.120" /> <!-- 120 mm -->
@@ -27,14 +27,13 @@
   <link name="base">
     <collision>
-      <origin xyz="0 0 ${wheel_rad - height_axis}" rpy="${PI/2} 0 ${PI/2}"/>
+      <origin xyz="0 0 0" rpy="${PI/2} 0 ${PI/2}"/>
       <geometry>
 				<mesh filename="package://prisme_description/meshes/simplified_body_v2.stl" scale="0.001 0.001 0.001"/>
-					<!--> <scale scale="1 .001 .001">1 0.001 0.001</scale> -->
       </geometry>
     </collision>
     <visual>
-      <origin xyz="0 0 0" rpy="${PI/2} 0 ${PI/2}"/>
+      <origin xyz="-${length/2} -${width/2+offset_side+wheel_thick/2+0.0025} -${0.020}" rpy="${PI/2} 0 ${PI/2}"/>
       <geometry>
-				<mesh filename="package://prisme_description/meshes/simplified_body_v2.stl" scale="0.001 0.001 0.001"/>
+				<mesh filename="package://prisme_description/meshes/body.stl" scale="0.001 0.001 0.001"/>
       </geometry>
       <material name="orange"/>
@@ -45,7 +44,7 @@
 			<!-- Fake values -->
       <inertia
-				ixx="1.0" ixy="0.0" ixz="0.0"
-	  		iyy="1.0" iyz="0.0"
-	  		izz="1.0"/>
+				ixx="0.001" ixy="0.0" ixz="0.0"
+	  		iyy="0.001" iyz="0.0"
+	  		izz="0.001"/>
     </inertial>
   </link>
@@ -60,8 +59,9 @@
 			</collision>
 			<visual>
-				<origin rpy="${reflect*PI/2} 0 0" />
+				<origin xyz="${wheel_rad} -${wheel_thick/2} -${wheel_rad}" rpy="0 0 ${PI/2}" />
 				<geometry>
-					<cylinder length="${wheel_thick}" radius="${wheel_rad}" />
+					<mesh filename="package://prisme_description/meshes/wheel.stl" scale="0.001 0.001 0.001"/>
 				</geometry>
+        <material name="blue"/>
 			</visual>
 		  <inertial>
@@ -70,7 +70,7 @@
 				<!-- Fake values -->
 		    <inertia
-					ixx="0.1" ixy="0.0" ixz="0.0"
-					iyy="0.1" iyz="0.0"
-					izz="0.1"/>
+					ixx="0.001" ixy="0.0" ixz="0.0"
+					iyy="0.001" iyz="0.0"
+					izz="0.001"/>
 		  </inertial>
 		</link>
@@ -93,10 +93,4 @@
 			</geometry>
 		</collision>
-		<visual>
-			<geometry>
-				<cylinder length="${caster_rod_length}" radius="${caster_sphere_rad/3}"/>
-			</geometry>
-      <material name="white"/>
-		</visual>
 	</link>
 	<!-- Caster rod Joint -->
@@ -113,10 +107,4 @@
 			</geometry>
 		</collision>
-		<visual>
-			<geometry>
-				<sphere radius="${caster_sphere_rad}"/>
-			</geometry>
-			<material name="white"/>
-		</visual>
 	</link>
 	<!-- Caster sphere Joint -->
@@ -133,10 +121,4 @@
 			</geometry>
 		</collision>
-		<visual>
-			<geometry>
-				<box size="${bpack_length} ${bpack_width} ${bpack_height}"/>
-			</geometry>
-      <material name="red"/>
-		</visual>
 	  <inertial>
 	    <origin xyz="0 0 0" rpy="0 0 0"/>
@@ -155,3 +137,24 @@
   	<origin xyz="${-(length/2 - bpack_offset - bpack_length/2)} 0 ${bpack_height/2}" rpy="0 0 0"/>
 	</joint>
+	<!-- IR Macro -->
+	<xacro:macro name="ir_front" params="position x y angle">
+		<link name="ir_front_${position}">
+			<!--
+			<visual>
+				<geometry>
+					<box size="0.007 0.010 0.005"/>
+				</geometry>
+				<material name="green"/>
+			</visual> -->
+		</link>
+		<joint name="joint_ir_front_${position}" type="fixed">
+			<parent link="base"/>
+			<child link="ir_front_${position}"/>
+			<origin xyz="${x} ${y} 0.018" rpy="0 0 ${angle}"/>
+		</joint>
+	</xacro:macro>
+	<xacro:ir_front position="left_center" x="0.05722" y="0.01804" angle="0.3054" /> <!-- 60cos(17.5)=57.22, 60sin(17.5)=18.04 -->
+	<xacro:ir_front position="right_center" x="0.05722" y="-0.01804" angle="-0.3054" />
+	<xacro:ir_front position="left" x="0.04424" y="0.04054" angle="0.7418" /> <!-- 60cos(42.5)=44.24, 60sin(42.5)=40.54 -->
+	<xacro:ir_front position="right" x="0.04424" y="-0.04054" angle="-0.7418" />
 </robot>

Commit message: Added macro for ir_front angles with Jade

File: prisme_description/urdf/prisme.xacro (robot description, xacro)
@@ -1,5 +1,4 @@
 <?xml version="1.0"?>
 <robot name="prisme" xmlns:xacro="http://www.ros.org/wiki/xacro">
-  <xacro:property name="PI" value="3.1415926535897931"/>
 	<!-- Fake values -->
   <xacro:property name="mass_body" value="0.300" />
@@ -20,4 +19,7 @@
 	<xacro:property name="bpack_offset" value="0.010" /> <!-- 10 mm -->
 	<xacro:property name="bpack_height" value="0.058" /> <!-- 58 mm -->
+	<xacro:property name="ir_front_rad" value="0.06" />
+	<xacro:property name="ir_angle1" value="${radians(17.5)}" />
+	<xacro:property name="ir_angle2" value="${radians(42.5)}" />
   <!-- Import all Gazebo-customization elements, including Gazebo colors -->
   <xacro:include filename="$(find prisme_description)/urdf/prisme.gazebo" />
@@ -27,5 +29,5 @@
   <link name="base">
     <collision>
-      <origin xyz="0 0 0" rpy="${PI/2} 0 ${PI/2}"/>
+      <origin xyz="0 0 0" rpy="${pi/2} 0 ${pi/2}"/>
       <geometry>
 				<mesh filename="package://prisme_description/meshes/simplified_body_v2.stl" scale="0.001 0.001 0.001"/>
@@ -33,5 +35,5 @@
     </collision>
     <visual>
-      <origin xyz="-${length/2} -${width/2+offset_side+wheel_thick/2+0.0025} -${0.020}" rpy="${PI/2} 0 ${PI/2}"/>
+      <origin xyz="-${length/2} -${width/2+offset_side+wheel_thick/2+0.0025} -${0.020}" rpy="${pi/2} 0 ${pi/2}"/>
       <geometry>
 				<mesh filename="package://prisme_description/meshes/body.stl" scale="0.001 0.001 0.001"/>
@@ -53,5 +55,5 @@
 		<link name="wheel_${side}">
 			<collision>
-				<origin rpy="${reflect*PI/2} 0 0" />
+				<origin rpy="${reflect*pi/2} 0 0" />
 				<geometry>
 					<cylinder length="${wheel_thick}" radius="${wheel_rad}" />
@@ -59,5 +61,5 @@
 			</collision>
 			<visual>
-				<origin xyz="${wheel_rad} -${wheel_thick/2} -${wheel_rad}" rpy="0 0 ${PI/2}" />
+				<origin xyz="${wheel_rad} -${wheel_thick/2} -${wheel_rad}" rpy="0 0 ${pi/2}" />
 				<geometry>
 					<mesh filename="package://prisme_description/meshes/wheel.stl" scale="0.001 0.001 0.001"/>
@@ -138,5 +140,5 @@
 	</joint>
 	<!-- IR Macro -->
-	<xacro:macro name="ir_front" params="position x y angle">
+	<xacro:macro name="ir_front" params="position angle">
 		<link name="ir_front_${position}">
 			<!--
@@ -151,10 +153,10 @@
 			<parent link="base"/>
 			<child link="ir_front_${position}"/>
-			<origin xyz="${x} ${y} 0.018" rpy="0 0 ${angle}"/>
+			<origin xyz="${ir_front_rad*cos(angle)} ${ir_front_rad*sin(angle)} 0.018" rpy="0 0 ${angle}"/>
 		</joint>
 	</xacro:macro>
-	<xacro:ir_front position="left_center" x="0.05722" y="0.01804" angle="0.3054" /> <!-- 60cos(17.5)=57.22, 60sin(17.5)=18.04 -->
-	<xacro:ir_front position="right_center" x="0.05722" y="-0.01804" angle="-0.3054" />
-	<xacro:ir_front position="left" x="0.04424" y="0.04054" angle="0.7418" /> <!-- 60cos(42.5)=44.24, 60sin(42.5)=40.54 -->
-	<xacro:ir_front position="right" x="0.04424" y="-0.04054" angle="-0.7418" />
+	<xacro:ir_front position="left_center" angle="${ir_angle1}" /> <!-- 60cos(17.5)=57.22, 60sin(17.5)=18.04 -->
+	<xacro:ir_front position="right_center" angle="${-ir_angle1}" />
+	<xacro:ir_front position="left" angle="${ir_angle2}" /> <!-- 60cos(42.5)=44.24, 60sin(42.5)=40.54 -->
+	<xacro:ir_front position="right" angle="${-ir_angle2}" />
 </robot>

Commit message: Integrated line-following sensors, improved inertial parameters

File: prisme_description/urdf/prisme.xacro (robot description, xacro)
@@ -22,4 +22,6 @@
 	<xacro:property name="ir_angle1" value="${radians(17.5)}" />
 	<xacro:property name="ir_angle2" value="${radians(42.5)}" />
+	<xacro:property name="ir_under_x" value="0.030" />
+	<xacro:property name="ir_under_y" value="0.008" />
   <!-- Import all Gazebo-customization elements, including Gazebo colors -->
   <xacro:include filename="$(find prisme_description)/urdf/prisme.gazebo" />
@@ -46,7 +48,7 @@
 			<!-- Fake values -->
       <inertia
-				ixx="0.001" ixy="0.0" ixz="0.0"
-	  		iyy="0.001" iyz="0.0"
-	  		izz="0.001"/>
+				ixx="${1e-3}" ixy="0.0" ixz="0.0"
+	  		iyy="${1e-3}" iyz="0.0"
+	  		izz="${1e-3}"/>
     </inertial>
   </link>
@@ -72,7 +74,7 @@
 				<!-- Fake values -->
 		    <inertia
-					ixx="0.001" ixy="0.0" ixz="0.0"
-					iyy="0.001" iyz="0.0"
-					izz="0.001"/>
+					ixx="${1e-4}" ixy="0.0" ixz="0.0"
+					iyy="${1e-4}" iyz="0.0"
+					izz="${1e-4}"/>
 		  </inertial>
 		</link>
@@ -82,5 +84,5 @@
     	<origin xyz="0 ${reflect*(width/2+offset_side+wheel_thick/2)} ${height_axis}" rpy="0 0 0"/>
     	<axis xyz="0 1 0"/>
-    	<dynamics damping="0.7"/>
+    	<dynamics damping="1"/>
   	</joint>
 	</xacro:macro>
@@ -128,7 +130,7 @@
 			<!-- Fake values -->
 	    <inertia
-				ixx="0.1" ixy="0.0" ixz="0.0"
-				iyy="0.1" iyz="0.0"
-				izz="0.1"/>
+				ixx="${1e-3}" ixy="0.0" ixz="0.0"
+				iyy="${1e-3}" iyz="0.0"
+				izz="${1e-3}"/>
 	  </inertial>
 	</link>
@@ -139,14 +141,13 @@
   	<origin xyz="${-(length/2 - bpack_offset - bpack_length/2)} 0 ${bpack_height/2}" rpy="0 0 0"/>
 	</joint>
-	<!-- IR Macro -->
+	<!-- IR front Macro -->
 	<xacro:macro name="ir_front" params="position angle">
 		<link name="ir_front_${position}">
-			<!--
-			<visual>
+			<!--visual>
 				<geometry>
 					<box size="0.007 0.010 0.005"/>
 				</geometry>
 				<material name="green"/>
-			</visual> -->
+			</visual-->
 		</link>
 		<joint name="joint_ir_front_${position}" type="fixed">
@@ -156,7 +157,25 @@
 		</joint>
 	</xacro:macro>
-	<xacro:ir_front position="left_center" angle="${ir_angle1}" /> <!-- 60cos(17.5)=57.22, 60sin(17.5)=18.04 -->
+	<xacro:ir_front position="left_center" angle="${ir_angle1}" />
 	<xacro:ir_front position="right_center" angle="${-ir_angle1}" />
-	<xacro:ir_front position="left" angle="${ir_angle2}" /> <!-- 60cos(42.5)=44.24, 60sin(42.5)=40.54 -->
+	<xacro:ir_front position="left" angle="${ir_angle2}" />
 	<xacro:ir_front position="right" angle="${-ir_angle2}" />
+	<!-- IR under Macro -->
+	<xacro:macro name="ir_under" params="position reflect">
+		<link name="ir_under_${position}">
+			<visual>
+				<geometry>
+					<box size="0.005 0.010 0.007"/>
+				</geometry>
+				<material name="green"/>
+			</visual>
+		</link>
+		<joint name="joint_ir_under_${position}" type="fixed">
+			<parent link="base"/>
+			<child link="ir_under_${position}"/>
+			<origin xyz="${ir_under_x} ${ir_under_y*reflect} 0" rpy="0 ${pi/2} 0"/>
+		</joint>
+	</xacro:macro>
+	<xacro:ir_under position="left" reflect="1" />
+	<xacro:ir_under position="right" reflect="-1" />
 </robot>

Commit message: Integrated linear camera module

File: prisme_description/urdf/prisme.xacro (robot description, xacro)
@@ -179,3 +179,18 @@
 	<xacro:ir_under position="left" reflect="1" />
 	<xacro:ir_under position="right" reflect="-1" />
+	<!-- Linear Camera Link -->
+	<link name="lc">
+		<visual>
+			<geometry>
+				<box size="0.01 0.017 0.017"/>
+			</geometry>
+			<material name="green"/>
+		</visual>
+	</link>
+	<!-- Linear Camera Joint -->
+	<joint name="joint_lc" type="fixed">
+  	<parent link="base"/>
+  	<child link="lc"/>
+  	<origin xyz="0.04 -0.008 0.065" rpy="0 0 0"/>
+	</joint>
 </robot>

Commit message: Integrated imu sensor (noise std tbd)

File: prisme_description/urdf/prisme.xacro (robot description, xacro)
@@ -181,10 +181,10 @@
 	<!-- Linear Camera Link -->
 	<link name="lc">
-		<visual>
+		<!--visual>
 			<geometry>
 				<box size="0.01 0.017 0.017"/>
 			</geometry>
 			<material name="green"/>
-		</visual>
+		</visual-->
 	</link>
 	<!-- Linear Camera Joint -->

Commit message: Optimized rates

File: prisme_description/urdf/prisme.xacro (robot description, xacro)
@@ -23,5 +23,5 @@
 	<xacro:property name="ir_angle2" value="${radians(42.5)}" />
 	<xacro:property name="ir_under_x" value="0.030" />
-	<xacro:property name="ir_under_y" value="0.008" />
+	<xacro:property name="ir_under_y" value="0.012" />
   <!-- Import all Gazebo-customization elements, including Gazebo colors -->
   <xacro:include filename="$(find prisme_description)/urdf/prisme.gazebo" />

Commit message: Fixed inertia

File: prisme_description/urdf/prisme.xacro (robot description, xacro)
@@ -3,6 +3,6 @@
 	<!-- Fake values -->
   <xacro:property name="mass_body" value="0.300" />
-	<xacro:property name="mass_wheel" value="0.05" />
-	<xacro:property name="mass_bpack" value="0.4" />
+	<xacro:property name="mass_wheel" value="0.025" />
+	<xacro:property name="mass_bpack" value="0.300" />
 	<xacro:property name="width" value="0.0936" /> <!-- 2*46.8 = 93.6 mm -->
 	<xacro:property name="length" value="0.120" /> <!-- 120 mm -->

Commit message: Fixed inertia and mass values

File: prisme_description/urdf/prisme.xacro (robot description, xacro)
@@ -46,9 +46,8 @@
       <origin xyz="0 0 ${height/2}" rpy="0 0 0"/>
       <mass value="${mass_body}"/>
-			<!-- Fake values -->
       <inertia
-				ixx="${1e-3}" ixy="0.0" ixz="0.0"
-	  		iyy="${1e-3}" iyz="0.0"
-	  		izz="${1e-3}"/>
+				ixx="${3e-4}" ixy="0.0" ixz="0.0"
+	  		iyy="${5e-4}" iyz="0.0"
+	  		izz="${6e-4}"/>
     </inertial>
   </link>
@@ -70,11 +69,10 @@
 			</visual>
 		  <inertial>
-		    <origin xyz="0 0 0" rpy="0 0 0"/> <!-- maybe wrong... -->
+		    <origin xyz="0 0 0" rpy="0 0 0"/>
 		    <mass value="${mass_wheel}"/>
-				<!-- Fake values -->
 		    <inertia
-					ixx="${1e-4}" ixy="0.0" ixz="0.0"
-					iyy="${1e-4}" iyz="0.0"
-					izz="${1e-4}"/>
+					ixx="${0.8e-5}" ixy="0.0" ixz="0.0"
+					iyy="${1.5e-5}" iyz="0.0"
+					izz="${0.8e-5}"/>
 		  </inertial>
 		</link>
@@ -85,4 +83,5 @@
     	<axis xyz="0 1 0"/>
     	<dynamics damping="1"/>
+    	<dynamics friction="1" damping="1.0"/>
   	</joint>
 	</xacro:macro>
@@ -126,11 +125,10 @@
 		</collision>
 	  <inertial>
-	    <origin xyz="0 0 0" rpy="0 0 0"/>
+	    <origin xyz="0.0 0.0 0.0" rpy="0 0 0"/>
 	    <mass value="${mass_bpack}"/>
-			<!-- Fake values -->
 	    <inertia
-				ixx="${1e-3}" ixy="0.0" ixz="0.0"
-				iyy="${1e-3}" iyz="0.0"
-				izz="${1e-3}"/>
+				ixx="${1.5e-4}" ixy="0.0" ixz="0.0"
+				iyy="${1e-4}" iyz="0.0"
+				izz="${0.7e-4}"/>
 	  </inertial>
 	</link>

Commit message: Integrated ros_control: transmission and dummy base link

File: prisme_description/urdf/prisme.xacro (robot description, xacro)
@@ -43,4 +43,6 @@
       <material name="orange"/>
     </visual>
+  </link>
+  <link name="base_dummy_inertia">
     <inertial>
       <origin xyz="0 0 ${height/2}" rpy="0 0 0"/>
@@ -51,5 +53,10 @@
 	  		izz="${6e-4}"/>
     </inertial>
-  </link>
+	</link>
+	<joint name="joint_base_dummy_inertia" type="fixed">
+  	<parent link="base"/>
+  	<child link="base_dummy_inertia"/>
+  	<origin xyz="0 0 0" rpy="0 0 0"/>
+	</joint>
 	<!-- Wheel Macro -->
 	<xacro:macro name="wheel" params="side reflect">
@@ -82,7 +89,19 @@
     	<origin xyz="0 ${reflect*(width/2+offset_side+wheel_thick/2)} ${height_axis}" rpy="0 0 0"/>
     	<axis xyz="0 1 0"/>
-    	<dynamics damping="1"/>
+			<limit
+				effort="100"
+				velocity="10" />
     	<dynamics friction="1" damping="1.0"/>
   	</joint>
+		<transmission name="trans_${side}">
+			<type>transmission_interface/SimpleTransmission</type>
+			<joint name="joint_${side}">
+				<hardwareInterface>VelocityJointInterface</hardwareInterface>
+			</joint>
+			<actuator name="motor_${side}">
+				<hardwareInterface>VelocityJointInterface</hardwareInterface>
+				<mechanicalReduction>1</mechanicalReduction>
+			</actuator>
+		</transmission>
 	</xacro:macro>
 	<!-- Wheels -->

Commit message: Removed former gazebo_ros_diff_drive plugin for the ros_control version

File: prisme_description/urdf/prisme.xacro (robot description, xacro)
@@ -11,7 +11,8 @@
 	<xacro:property name="offset_side" value="0.002" /> <!-- 2 mm -->
 	<xacro:property name="wheel_thick" value="0.008" /> <!-- 8 mm -->
-	<xacro:property name="wheel_rad" value="0.035" /> <!-- 35 mm -->
+	<xacro:property name="wheel_radius" value="0.035" /> <!-- 35 mm -->
+	<xacro:property name="wheel_separation" value="${width+2*offset_side+wheel_thick}"/>
 	<xacro:property name="caster_sphere_rad" value="0.006" /> <!-- 6 mm -->
-	<xacro:property name="caster_rod_length" value="${(wheel_rad-height_axis)-2*caster_sphere_rad}" />
+	<xacro:property name="caster_rod_length" value="${(wheel_radius-height_axis)-2*caster_sphere_rad}" />
 	<xacro:property name="caster_offset" value="0.045" /> <!-- 45 mm -->
 	<xacro:property name="bpack_length" value="0.028" /> <!-- 28 mm -->
@@ -65,9 +66,9 @@
 				<origin rpy="${reflect*pi/2} 0 0" />
 				<geometry>
-					<cylinder length="${wheel_thick}" radius="${wheel_rad}" />
+					<cylinder length="${wheel_thick}" radius="${wheel_radius}" />
 				</geometry>
 			</collision>
 			<visual>
-				<origin xyz="${wheel_rad} -${wheel_thick/2} -${wheel_rad}" rpy="0 0 ${pi/2}" />
+				<origin xyz="${wheel_radius} -${wheel_thick/2} -${wheel_radius}" rpy="0 0 ${pi/2}" />
 				<geometry>
 					<mesh filename="package://prisme_description/meshes/wheel.stl" scale="0.001 0.001 0.001"/>
